Commit message: fixed typo in joint name

File: motoman_ar1440e_support/urdf/ar1440e_macro.xacro (robot description, xacro)
@@ -161,5 +161,5 @@
       <axis xyz="0 0 1" />
     </joint>
-    <joint name="${prefix}joint_4u" type="revolute">
+    <joint name="${prefix}joint_4_u" type="revolute">
       <parent link="${prefix}link_3_l2" />
       <child link = "${prefix}link_4_u" />

Commit message: renamed tcp_link to tool0

File: motoman_ar1440e_support/urdf/ar1440e_macro.xacro (robot description, xacro)
@@ -2,4 +2,9 @@
 <robot xmlns:xacro="http://ros.org/wiki/xacro">
   <xacro:macro name="motoman_ar1440e" params="prefix">
+    <!-- Properties -->
+    <material name="yaskawa_blue">
+          <color rgba="0.12941 0.14902 0.74902 1" />
+    </material>
+    <!-- link list -->
     <link name="${prefix}base_link" >
       <visual>
@@ -138,6 +143,6 @@
       </collision>
     </link>
-   <link name="${prefix}tcp_link" />
-<!-- WARNING: effort fields have not been set -->
+   <link name="${prefix}tool0" />
+    <!-- end of link list -->
    <joint name="${prefix}joint_1_s" type="revolute">
       <parent link="${prefix}base_link" />
@@ -189,8 +194,16 @@
       <axis xyz="0 0 1" />
     </joint>
-    <joint name="${prefix}tcp_joint" type="fixed">
-      <parent link="${prefix}link_7_t" />
-      <child link = "${prefix}tcp_link" />
-      <origin xyz="0 0 0.006" rpy="0 0 0" />
+    <joint name="${prefix}joint_7_t-tool0" type="fixed">
+        <origin xyz="0 0 0" rpy="0 0 0"/>
+        <parent link="${prefix}link_7_t"/>
+        <child link="${prefix}tool0"/>
+    </joint>
+    <!-- end of joint list -->
+    <!-- ROS base_link to Robot Manufacturer World Coordinates transform -->
+    <link name="${prefix}base" />
+    <joint name="${prefix}base_link-base" type="fixed">
+        <origin xyz="0 0 0.540" rpy="0 0 0"/>
+        <parent link="${prefix}base_link"/>
+        <child link="${prefix}base"/>
     </joint>
   </xacro:macro>

Commit message: fixed import bug by adding prefix to color macro

File: motoman_ar1440e_support/urdf/ar1440e_macro.xacro (robot description, xacro)
@@ -3,5 +3,5 @@
   <xacro:macro name="motoman_ar1440e" params="prefix">
     <!-- Properties -->
-    <material name="yaskawa_blue">
+    <material name="${prefix}yaskawa_blue">
           <color rgba="0.12941 0.14902 0.74902 1" />
     </material>
